File: hardware/KiCad/thundervolt_1/thundervolt_hw1.kicad_sch (KiCad schematic)
At the start: 59 parts, among them U1 TPS628681ARQYR, U2 TPS628681ARQYR, U3 TPS628682ARQYR, U4 TPS63810YFFR, U5 ATTINY1616-MNR, U6 LP5907UVX-1.8_NOPB, U7 TMP1075NDRLR

Commit message: U10 FET Mode
Parts:
- removed R6: 0Ω, Resistor_SMD:R_0402_1005Metric, symbol Device:R_Small
- added Q1: NX7002BKMYL, Package_DFN_QFN:Diodes_DFN1006-3, symbol Transistor_FET:DMG2302U
- D1: footprint LED_SMD:LED_0402_1005Metric -> SamacSys_Parts:LED_0603_1608Metric
Connections:
- net GND: now also U5.8 (PA7), Q1.2 (S)
- net U10: now also Q1.3 (D); no longer U5.11 (PB3)
- net at U5.15 (PC0): now also D1.2 (A)
- new net: Q1.1 (G), U5.11 (PB3)
- no-connect marks 10 -> 9
Other:
- moved on the sheet: TP6
