File: hardware/KiCad/thundervolt_lite/thundervolt_lite.kicad_sch (KiCad schematic)
At the start: 59 parts, among them U1 TPS628681ARQYR, U2 TPS628681ARQYR, U3 TPS628682ARQYR, U4 TPS63810YFFR, U5 ATTINY1616-MNR, U7 TMP1075NDRLR, U8 MIC5365-1.8YC5-TR

Commit message: U10 FET Mode
Parts:
- removed R6: 0Ω, Resistor_SMD:R_0402_1005Metric, symbol Device:R_Small
- added Q1: PJE8408_R1_00001, Package_TO_SOT_SMD:SOT-523, symbol Transistor_FET:DMN10H700S
Connections:
- net GND: now also U5.8 (PA7), Q1.2 (S)
- net U10: now also Q1.3 (D); no longer U5.11 (PB3)
- net at U5.15 (PC0): now also D1.2 (A)
- new net: Q1.1 (G), U5.11 (PB3)
- no-connect marks 10 -> 9
Other:
- moved on the sheet: TP6
